Commit message: removi o pacote da camera e ajustei as transformações do LIDAR

File: calman_description/description/lidar.xacro (robot description, xacro)
@@ -4,5 +4,5 @@
         <parent link="chassis"/>
         <child link="laser_frame"/>
-        <origin xyz="0.0 0 0.165" rpy="0 0 ${pi/2}"/>
+        <origin xyz="0.018 0.0 0.19" rpy="0.0 0.0 0.0"/>
     </joint>
     <link name="laser_frame">

Commit message: corrigir a orientacao do lidar

File: calman_description/description/lidar.xacro (robot description, xacro)
@@ -4,5 +4,5 @@
         <parent link="chassis"/>
         <child link="laser_frame"/>
-        <origin xyz="0.018 0.0 0.19" rpy="0.0 0.0 0.0"/>
+        <origin xyz="0.018 0.0 0.19" rpy="0.0 0.0 ${pi}"/>
     </joint>
     <link name="laser_frame">
@@ -19,5 +19,5 @@
         </collision>
         <xacro:inertial_cylinder mass="0.05" length="0.04" radius="0.0325">
-            <origin xyz="0 0 0" rpy="0 0 0"/>
+            <origin xyz="0.018 0 0.19" rpy="0 0 ${pi}"/>
         </xacro:inertial_cylinder>
     </link>
